File: pcb/LCR_measurement.kicad_sch (KiCad schematic)
At the start: 51 parts, among them J3 Conn_01x04_Socket, J4 Conn_01x01_Pin, J5 Conn_01x01_Pin, SW2 SW_DIP_x02, SW3 SW_SPST, U3 AT24CM02-SSHM, U4 ATtiny1604-SS, U5 FT230XS, U6 MCP4921, U7 MCP6001-OT, U8 MCP3562RT-E/ST

Commit message: Fix wrong part number
Parts:
- U6: DigiKey MCP4921T-E/MSCT-ND -> MCP4921T-E/SNCT-ND
Changed lines of the file:
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@@
 			)
 		)
-		(property "DigiKey" "MCP4921T-E/MSCT-ND"
+		(property "DigiKey" "MCP4921T-E/SNCT-ND"
 			(at 160.02 115.57 0)
 			(effects
